File: 0007_Relay_Module_ALQ105.kicad_sch (KiCad schematic)
At the start: 16 parts, among them J1 Screw_Terminal_01x03, J2 Screw_Terminal_01x03, K1 ALQ105, K2 ALQ105, Q1 BC817, Q2 BC817, U1 TLP185, U2 TLP185

Commit message: Add files via upload
Parts:
- added D5: LED, LED_SMD:LED_0805_2012Metric, symbol Device:LED
- added R5: 470r, Resistor_SMD:R_0805_2012Metric, symbol Device:R
- added U3: ~, Moduler_:pin_header_5-3, symbol moduler_pin:air
- J1, J2: footprint (none) -> TerminalBlock_4Ucon:TerminalBlock_4Ucon_1x03_P3.50mm_Horizontal
- K1, K2: footprint ALQ105 -> ALQ105:ALQ105
Connections:
- net +5V: now also R5.1, U3.7
- net GND: now also D5.1 (K), U3.9
- net R1: now also U3.12
- net R2: now also U3.13
- new net: D5.2 (A), R5.2
- no-connect marks 0 -> 14
Other:
- note added: "AIR PIN"
- note added: "RELAY"
- moved on the sheet: D1, D2, D3, D4, J1, J2, K1, K2, Q1, Q2, R1, R2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
